File: pcb/dabao-choc/dabao-choc.kicad_pcb (KiCad board)
At the start: 2 copper layers, 257.4 x 105.6 mm, 91 parts, among them J1 USB_C_Receptacle_USB2.0_16P, J2 USB_C_Receptacle_USB2.0_16P, J3 Conn_01x04_Pin, J4 Conn_01x04_Pin, J5 Conn_Battery, SW1 SW_RESET, SW2 SW_POWER, U1 nice_nano, U2 MCP23017_SP

Commit message: Add trackpoint parts
Parts:
- added J6: MJ-4PP-9, Library:TPSensorModule_Connector, F.Cu at (239.0, 141.6)
- added REF**: TPSensorModule, Library:TPSensorModule, F.Cu at (270.2, 118.5)
- added U3: MCP23017_SO, Package_SO:SOIC-28W_7.5x17.9mm_P1.27mm, B.Cu at (236.9, 139.7)
- U2: moved to B.Cu
- moved U2 57.7 mm to (239.8, 138.1), turned to 180 degrees
- moved SW1 27.6 mm to (233.0, 102.5)
- moved J5 15.9 mm to (248.2, 121.5), turned to 180 degrees
- moved J1 4.25 mm to (228.8, 152.0)
- moved J2 3.95 mm to (210.1, 158.0)
- moved U1 2.95 mm to (232.9, 111.9)
- moved J3 1.19 mm to (225.0, 141.4)
- moved J4 1.19 mm to (214.0, 133.9)
Connections:
- net /BAT+ renamed Net-(SW2-A)
- net /RST renamed Net-(U1-RST)
Other:
- board size 257.4 x 105.6 mm -> 259.3 x 107.8 mm
