File: pcb/dabao-choc/dabao-choc.kicad_sch (KiCad schematic)
At the start: 81 parts, among them J1 USB_C_Receptacle_USB2.0_16P, J2 USB_C_Receptacle_USB2.0_16P, J3 Conn_01x04_Pin, J4 Conn_01x04_Pin, J5 Conn_Battery, SW1 SW_RESET, SW2 SW_POWER, U1 nice_nano, U2 MCP23017_SP

Commit message: Add trackpoint parts
Parts:
- added J6: MJ-4PP-9, Library:TPSensorModule_Connector, symbol TPS42:MJ-4PP-9
- added U3: MCP23017_SO, Package_SO:SOIC-28W_7.5x17.9mm_P1.27mm, symbol Interface_Expansion:MCP23017_SO
Connections:
- net SCK: now also J2.A6 (D+), J2.B6 (D+), J4.3 (Pin_3), U2.12 (SCK)
- net SDA: now also J2.A7 (D-), J2.B7 (D-), J4.2 (Pin_2), U2.13 (SDA)
Changed lines of the file:
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@@
 		)
 	)
+	(label "SCK"
+		(at 83.82 115.57 180)
+		(effects
+			(font
+				(size 1.27 1.27)
+			)
+			(justify right bottom)
+		)
+	)
 	(label "rowR_home"
 		(at 161.29 58.42 0)
@@
 		)
 	)
+	(label "SDA"
+		(at 83.82 113.03 180)
+		(effects
+			(font
+				(size 1.27 1.27)
+			)
+			(justify right bottom)
+		)
+	)
 	(label "colR_ring"
 		(at 200.66 143.51 180)
@@
 	)
 	(symbol
+		(lib_id "Interface_Expansion:MCP23017_SO")
+		(at 54.61 191.77 0)
+		(unit 1)
+		(exclude_from_sim no)
+		(in_bom yes)
+		(on_board yes)
+		(dnp no)
+		(fields_autoplaced yes)
+		(property "Reference" "U3"
+			(at 56.7533 163.83 0)
+			(effects
+				(font
+					(size 1.27 1.27)
+				)
+				(justify left)
+			)
+		)
+		(property "Value" "MCP23017_SO"
+			(at 56.7533 166.37 0)
+			(effects
+				(font
+					(size 1.27 1.27)
+				)
+				(justify left)
+			)
+		)
+		(property "Footprint" "Package_SO:SOIC-28W_7.5x17.9mm_P1.27mm"
+			(at 59.69 217.17 0)
+			(effects
+				(font
+					(size 1.27 1.27)
+				)
+				(justify left)
+				(hide yes)
+			)
+		)
+		(property "Datasheet" "https://ww1.microchip.com/downloads/aemDocuments/documents/APID/ProductDocuments/DataSheets/MCP23017-Data-Sheet-DS20001952.pdf"
+			(at 59.69 219.71 0)
+			(effects
+				(font
+					(size 1.27 1.27)
+				)
+				(justify left)
+				(hide yes)
+			)
+		)
+		(property "Description" "16-bit I/O expander, I2C, interrupts, w pull-ups, GPA/B7 output only (https://microchip.my.site.com/s/article/GPA7---GPB7-Cannot-Be-Used-as-Inputs-In-MCP23017),  SOIC-28"
+			(at 54.61 191.77 0)
+			(effects
+				(font
+					(size 1.27 1.27)
+				)
+				(hide yes)
+			)
+		)
+		(pin "12"
+		)
+		(pin "19"
+		)
+		(pin "13"
+		)
+		(pin "1"
+		)
+		(pin "2"
+		)
+		(pin "3"
+		)
+		(pin "4"
+		)
+		(pin "5"
+		)
+		(pin "6"
+		)
+		(pin "7"
+		)
+		(pin "8"
+		)
+		(pin "21"
+		)
+		(pin "22"
+		)
+		(pin "23"
+		)
+		(pin "17"
+		)
+		(pin "16"
+		)
+		(pin "15"
+		)
+		(pin "11"
+		)
+		(pin "14"
+		)
+		(pin "20"
+		)
+		(pin "18"
+		)
+		(pin "9"
+		)
+		(pin "10"
+		)
+		(pin "24"
+		)
+		(pin "25"
+		)
+		(pin "26"
+		)
+		(pin "27"
+		)
+		(pin "28"
+		)
+		(instances
+			(project ""
+				(path "/f7dfc45c-83ad-43c7-9815-463af0b28fbd"
+					(reference "U3")
+					(unit 1)
+				)
+			)
+		)
+	)
+	(symbol
 		(lib_id "PCM_marbastlib-choc:choc_v1_SW_HS_CPG135001S30")
 		(at 125.73 31.75 0)
@@
 					(unit 1)
 				)
+			)
+		)
+	)
+	(symbol
+		(lib_id "TPS42:MJ-4PP-9")
+		(at 229.87 83.82 0)
+		(unit 1)
+		(exclude_from_sim no)
+		(in_bom yes)
+		(on_board yes)
+		(dnp no)
+		(property "Reference" "J6"
+			(at 228.6 73.66 0)
+			(effects
+				(font
+					(size 1.524 1.524)
+				)
+			)
+		)
+		(property "Value" "MJ-4PP-9"
+			(at 228.6 76.2 0)
+			(effects
+				(font
+					(size 1.524 1.524)
+				)
+			)
+		)
+		(property "Footprint" "Library:TPSensorModule_Connector"
+			(at 229.87 77.724 0)
+			(effects
+				(font
+					(size 1.524 1.524)
+				)
+			)
+		)
+		(property "Datasheet" ""
+			(at 229.87 83.82 0)
+			(effects
+				(font
+					(size 1.524 1.524)
+				)
+			)
+		)
+		(property "Description" ""
+			(at 229.87 83.82 0)
+			(effects
+				(font
+					(size 1.27 1.27)
+				)
+				(hide yes)
+			)
+		)
+		(pin "3"
+		)
+		(pin "4"
+		)
+		(pin "1"
+		)
+		(pin "2"
+		)
+		(instances
+			(project ""
+				(path "/f7dfc45c-83ad-43c7-9815-463af0b28fbd"
+					(reference "J6")
+					(unit 1)
+				)
